File: HW/AD4630 breakout.kicad_pcb (KiCad board)
At the start: 4 copper layers, 45 x 50 mm, 33 parts, among them J1 IN0, J2 IN1, J3 Conn_02x09_Counter_Clockwise, J4 IN0, U1 AD4630-24BBCZ, U2 AMS1117-1.8, U3 TXS0108EPW, U4 TXS0108EPW, U6 LTC6655

Commit message: updated PCB
Parts:
- removed H1, H2, H3, H4: MountingHole, MountingHole:MountingHole_3.2mm_M3_Pad_Via
- removed kibuzzard-638251C8: G***, kibuzzard-638251C8
- removed kibuzzard-638251EC: G***, kibuzzard-638251EC
- J3: value Conn_02x09_Counter_Clockwise -> IO
Connections:
- J3 pad 17: +3V3 -> +5V
Routing:
- added copper zone on In1.Cu, net +5V
Other:
- board size 45 x 50 mm -> 35 x 48 mm
- board text added: "5V"
- board text added: "ADA4630 Breakout NNNI 0123"
