File: HW/AD4630 breakout.kicad_sch (KiCad schematic)
At the start: 1 part, among them U1 AD4630-24BBCZ

Commit message: Updated PCB
Parts:
- added U2: AMS1117-1.8, Package_TO_SOT_SMD:SOT-89-3, symbol Regulator_Linear:AMS1117-1.8
- added U3, U4: TXS0108EPW, Package_SO:TSSOP-20_4.4x6.5mm_P0.65mm, symbol Logic_LevelTranslator:TXS0108EPW
- added U5: Pico, RPi_Pico:RPi_Pico_SMD_TH, symbol MCU_RaspberryPi_and_Boards:Pico
Connections:
- net +5V: now reaches U1.A3 (VDD_5V)
- net +5V: now also U1.B3 (VDD_5V), U1.B8 (VIO)
- net +1V8: now reaches U1.A8 (VIO)
- net +1V8: now also U1.G3 (VDD_1-8V), U1.H3 (VDD_1-8V_2)
Other:
- moved on the sheet: U1A, U1B

Commit message: PCB updated
Parts:
- added C1, C11, C12, C2, C3, C4: 10uF, Capacitor_SMD:C_0603_1608Metric, symbol Device:C_Small
- added C10, C5, C6, C7, C8, C9: C, Capacitor_SMD:C_0603_1608Metric, symbol Device:C_Small
- added J1: IN0, Connector_PinHeader_2.54mm:PinHeader_1x02_P2.54mm_Vertical, symbol Connector_Generic:Conn_01x02
- added J2: IN1, Connector_PinHeader_2.54mm:PinHeader_1x02_P2.54mm_Vertical, symbol Connector_Generic:Conn_01x02
- added J3, J4: IO, Connector_PinHeader_2.54mm:PinHeader_1x09_P2.54mm_Vertical, symbol Connector_Generic:Conn_01x09
- added R1, R2, R3, R4: R, Resistor_SMD:R_0603_1608Metric, symbol Device:R
- added U6: LTC6655BHLS8-5-PBF, LTC6655:LTC6655BHLS8-5-PBF, symbol LTC6655:LTC6655BHLS8-5-PBF
Connections:
- net +1V8: now also U1.B8 (VIO), U2.2 (VO), U3.2 (VCCA), U4.2 (VCCA), C1.1, C12.1, C2.1
- net +5V: now also U2.3 (VI), U3.19 (VCCB), U4.19 (VCCB), C11.1, C3.1, C4.1; no longer U1.B8 (VIO)
- net GND: now also U2.1 (GND), U3.11 (GND), U4.11 (GND), C1.2, C10.1, C11.2, C12.2, C2.2, C3.2, C4.2, C7.2, C8.1, C9.2
- net SDO6: now reaches U4.1 (A1)
- net SDO6: now also U1.F7 (SDO6)
- net OE1: now reaches U4.10 (OE)
- net OE1: now also J4.1 (Pin_1)
- net at U4.12 (B8): now also J4.9 (Pin_9)
- net at U4.13 (B7): now also J4.8 (Pin_8)
- net at U4.14 (B6): now also J4.7 (Pin_7)
- net at U4.15 (B5): now also J4.6 (Pin_6)
- net at U4.16 (B4): now also J4.5 (Pin_5)
- net at U4.17 (B3): now also J4.4 (Pin_4)
- net at U4.18 (B2): now also J4.3 (Pin_3)
- net at U4.20 (B1): now also J4.2 (Pin_2)
- net SDO4: now reaches U4.3 (A2)
- net SDO4: now also U1.F8 (SDO4)
- net SDO7: now reaches U4.4 (A3)
- net SDO7: now also U1.G7 (SDO7)
- net SDO5: now reaches U4.5 (A4)
- net SDO5: now also U1.G8 (SDO5)
- net SCK: now reaches U4.6 (A5)
- net SCK: now also U1.H7 (SCK)
- net SDI: now reaches U4.7 (A6)
- net SDI: now also U1.H6 (SDI)
- net CS: now reaches U4.8 (A7)
- net CS: now also U1.H5 (CS)
- net REFIN: now reaches U1.A2 (REFIN)
- net CNV: now reaches U1.A6 (CNV)
- net CNV: now also U3.1 (A1)
- net RST: now reaches U1.A7 (RST)
- net RST: now also U3.3 (A2)
- net IN0+: now reaches U1.B1 (IN0+)
- net IN0+: now also C5.1, C7.1, R1.2
- net IN0-: now reaches U1.C1 (IN0)
- net IN0-: now also C5.2, C8.2, R2.2
- net SDO3: now reaches U1.C7 (SDO3)
- net SDO3: now also U3.5 (A4)
- net SDO1: now reaches U1.C8 (SDO1)
- net SDO1: now also U3.4 (A3)
- net REF: now reaches U1.D2 (REF)
- net REF: now also U1.D3 (REF), U1.E2 (REF), U1.E3 (REF)
- net SDO2: now reaches U1.D7 (SDO2)
- net SDO2: now also U3.7 (A6)
- net SDO0: now reaches U1.D8 (SDO0)
- net SDO0: now also U3.6 (A5)
- net SCK OUT: now reaches U1.E8 (BUSY_SCKOUT)
- net SCK OUT: now also U3.8 (A7)
- net IN1+: now reaches U1.F1 (IN1+)
- net IN1+: now also C6.1, C9.1, R3.2
- net IN1-: now reaches U1.G1 (IN1)
- net IN1-: now also C10.2, C6.2, R4.2
- net OE: now reaches U3.10 (OE)
- net OE: now also J3.1 (Pin_1)
- net at U3.12 (B8): now also J3.9 (Pin_9)
- net at U3.13 (B7): now also J3.8 (Pin_8)
- net at U3.14 (B6): now also J3.7 (Pin_7)
- net at U3.15 (B5): now also J3.6 (Pin_6)
- net at U3.16 (B4): now also J3.5 (Pin_5)
- net at U3.17 (B3): now also J3.4 (Pin_4)
- net at U3.18 (B2): now also J3.3 (Pin_3)
- net at U3.20 (B1): now also J3.2 (Pin_2)
- new net: J2.2 (Pin_2), R4.1
- new net: J1.1 (Pin_1), R1.1
- new net: J1.2 (Pin_2), R2.1
- new net: J2.1 (Pin_1), R3.1
- no-connect marks 0 -> 2
Other:
- moved on the sheet: U2, U3, U4

Commit message: Updated PCB
Parts:
- removed J3, J4: IO, Connector_PinHeader_2.54mm:PinHeader_1x09_P2.54mm_Vertical, symbol Connector_Generic:Conn_01x09
- removed U5: Pico, RPi_Pico:RPi_Pico_SMD_TH, symbol MCU_RaspberryPi_and_Boards:Pico
- added C13, C14: 10uF, Capacitor_SMD:C_0603_1608Metric, symbol Device:C_Small
- added J3: Conn_02x09_Counter_Clockwise, Connector_PinHeader_2.54mm:PinHeader_2x09_P2.54mm_Vertical, symbol Connector_Generic:Conn_02x09_Counter_Clockwise
- U6: value LTC6655BHLS8-5-PBF -> LTC6655
Connections:
- net GND: now also U6.3 (GND), U6.4 (GND), U6.5 (GND), U6.8 (GND), C13.2, C14.2
- net OE: now also J3.1 (Pin_1)
- net OE1: now also J3.10 (Pin_10)
- net REFIN: now also U6.6 (VOUT_S), U6.7 (VOUT_F), C14.1
- net at U4.12 (B8): now also J3.18 (Pin_18)
- net at U4.13 (B7): now also J3.17 (Pin_17)
- net at U4.14 (B6): now also J3.16 (Pin_16)
- net at U4.15 (B5): now also J3.15 (Pin_15)
- net at U4.16 (B4): now also J3.14 (Pin_14)
- net at U4.17 (B3): now also J3.13 (Pin_13)
- net at U4.18 (B2): now also J3.12 (Pin_12)
- net at U4.20 (B1): now also J3.11 (Pin_11)
- net at U3.12 (B8): now also J3.9 (Pin_9)
- net at U3.13 (B7): now also J3.8 (Pin_8)
- net at U3.14 (B6): now also J3.7 (Pin_7)
- net at U3.15 (B5): now also J3.6 (Pin_6)
- net at U3.16 (B4): now also J3.5 (Pin_5)
- net at U3.17 (B3): now also J3.4 (Pin_4)
- net at U3.18 (B2): now also J3.3 (Pin_3)
- net at U3.20 (B1): now also J3.2 (Pin_2)
- net at U6.1 (~{SHDN}): now also U6.2 (VIN), C13.1
Other:
- note added: "yneos?"

Commit message: Finished PCB
Parts:
- added H1, H2, H3, H4: MountingHole, MountingHole:MountingHole_3.2mm_M3_Pad_Via, symbol Mechanical:MountingHole
- added J4: IN0, Connector_PinHeader_2.54mm:PinHeader_1x02_P2.54mm_Vertical, symbol Connector_Generic:Conn_01x02
Connections:
- net +1V8: now also U3.10 (OE), U4.10 (OE)
- net +5V: no longer C11.1, C3.1, C4.1, U2.3 (VI), U3.19 (VCCB), U4.19 (VCCB)
- net GND: now also J3.10 (Pin_10), J3.8 (Pin_8), J4.2 (Pin_2)
- net REFIN: now also J4.1 (Pin_1)
- net SDO4/: now reaches J3.11 (Pin_11)
- net SDO4/: now also U4.18 (B2); no longer U4.20 (B1)
- net SDO6/: now reaches J3.12 (Pin_12)
- net SDO6/: now also U4.20 (B1); no longer U4.18 (B2)
- net SDO5/: now reaches J3.13 (Pin_13)
- net SDO5/: now also U4.16 (B4); no longer U4.17 (B3)
- net SDO7/: now reaches J3.14 (Pin_14)
- net SDO7/: now also U4.17 (B3); no longer U4.16 (B4)
- net SCK/: now reaches U4.15 (B5)
- net SCK/: now also J3.16 (Pin_16); no longer J3.15 (Pin_15)
- net SDI/: now reaches U4.14 (B6)
- net SDI/: now also J3.15 (Pin_15); no longer J3.16 (Pin_16)
- net +3V3: now reaches J3.17 (Pin_17)
- net +3V3: now also C11.1, C3.1, C4.1, J3.9 (Pin_9), U2.3 (VI), U3.19 (VCCB), U4.19 (VCCB); no longer U4.13 (B7)
- net at U4.12 (B8): no longer J3.18 (Pin_18)
- net CNV/: now reaches U3.20 (B1)
- net CNV/: now also J3.1 (Pin_1); no longer J3.2 (Pin_2)
- net RST/: now reaches U3.18 (B2)
- net RST/: now also J3.2 (Pin_2); no longer J3.3 (Pin_3)
- net SDO1/: now reaches U3.17 (B3)
- net SDO1/: now also J3.3 (Pin_3); no longer J3.4 (Pin_4)
- net SDO0/: now reaches J3.5 (Pin_5)
- net SDO0/: now also U3.15 (B5); no longer U3.16 (B4)
- net SDO2/: now reaches J3.6 (Pin_6)
- net SDO2/: now also U3.14 (B6); no longer U3.15 (B5)
- net SCKo/: now reaches J3.7 (Pin_7)
- net SCKo/: now also U3.13 (B7); no longer U3.14 (B6)
- net at U3.12 (B8): no longer J3.9 (Pin_9)
- removed net OE: J3.1 (Pin_1), U3.10 (OE)
- removed net OE1: J3.10 (Pin_10), U4.10 (OE)
- new net CS/: J3.18 (Pin_18), U4.13 (B7)
- new net SDO3/: J3.4 (Pin_4), U3.16 (B4)
- no-connect marks 2 -> 4
Other:
- moved on the sheet: J3

Commit message: updated PCB
Parts:
- removed H1, H2, H3, H4: MountingHole, MountingHole:MountingHole_3.2mm_M3_Pad_Via, symbol Mechanical:MountingHole
- J3: value Conn_02x09_Counter_Clockwise -> IO
Connections:
- net +3V3: no longer J3.17 (Pin_17)
- net +5V: now also J3.17 (Pin_17)
Other:
- moved on the sheet: U1B
