File: Hardware/AD4630 breakout.kicad_pcb (KiCad board)
At the start: 4 copper layers, 35 x 48 mm, 27 parts, among them J1 IN0, J2 IN1, J3 IO, J4 IN0, U1 AD4630-24BBCZ, U2 AMS1117-1.8, U3 TXS0108EPW, U4 TXS0108EPW, U6 LTC6655

Commit message: updated files
Parts:
- removed J3: IO, Connector_PinHeader_2.54mm:PinHeader_2x09_P2.54mm_Vertical
- moved C13 25.3 mm to (107.0, 95.8)
- moved C14 25.3 mm to (107.0, 88.2)
- moved U6 25.3 mm to (107.0, 92.0)
- moved C1 21.3 mm to (164.2, 83.4)
- moved C3 21.3 mm to (164.2, 79.0)
- moved C11 18.2 mm to (172.8, 89.8)
- moved C12 18.2 mm to (172.8, 96.2)
- moved U2 18.2 mm to (172.0, 93.0)
- moved C2 17.5 mm to (117.2, 86.4)
- moved C4 17.5 mm to (117.2, 82.0)
- moved U3 6.08 mm to (133.0, 87.0), turned to 135 degrees
- moved U4 3.35 mm to (151.0, 87.0), turned to 45 degrees
- moved C6 0.80 mm to (145.2, 106.0)
- moved C7 0.80 mm to (137.6, 103.8)
- moved J4 0.80 mm to (134.3, 114.8)
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Connections:
- U3 pad 1: /CNV -> unconnected-(U3-Pad1)
- U3 pad 3: /RST -> unconnected-(U3-Pad3)
- U3 pad 4: /SDO1 -> unconnected-(U3-Pad4)
- U3 pad 5: /SDO3 -> unconnected-(U3-Pad5)
- U3 pad 6: /SDO0 -> unconnected-(U3-Pad6)
- U3 pad 7: /SDO2 -> unconnected-(U3-Pad7)
- U3 pad 8: /SCK OUT -> unconnected-(U3-Pad8)
- U4 pad 1: /SDO6 -> unconnected-(U4-Pad1)
- U4 pad 3: /SDO4 -> unconnected-(U4-Pad3)
- U4 pad 4: /SDO7 -> unconnected-(U4-Pad4)
- U4 pad 5: /SDO5 -> unconnected-(U4-Pad5)
- U4 pad 6: /SCK -> unconnected-(U4-Pad6)
- U4 pad 7: /SDI -> unconnected-(U4-Pad7)
- U4 pad 8: /CS -> unconnected-(U4-Pad8)
Routing:
- net +3V3: track 0.00 -> 9.46 mm, vias 3 -> 1
- net /RST/: track 11.7 -> 5.12 mm
- net /CS/: track 10.1 -> 4.29 mm
- net /SDO6/: track 9.68 -> 4.34 mm
- net /CNV/: track 8.93 -> 3.75 mm
- net /CNV: track 8.86 -> 4.73 mm
- net /CS: track 9.81 -> 5.70 mm
- net /SDI: track 8.66 -> 4.73 mm
- net /SCK/: track 9.55 -> 5.66 mm
- net /SDO2/: track 9.69 -> 5.98 mm
- net /RST: track 7.39 -> 3.77 mm
- net /SDO3: track 7.26 -> 3.77 mm
- net /SDO1: track 6.39 -> 2.90 mm
- net /SDO0: track 6.21 -> 2.80 mm
- net /SCK: track 7.04 -> 3.77 mm
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- removed copper zone on In2.Cu, net +1V8
- removed copper zone on In2.Cu, net +3V3
- removed copper zone on In1.Cu, net +5V
- removed copper zone on B.Cu, net GND
- removed copper zone on In1.Cu, net GND
- removed copper zone on In2.Cu, net GND
Other:
- board size 35 x 48 mm -> 35 x 40 mm
- board text added: "AD4630 Breakout NNNI 0123"
- board text removed: "ADA4630 Breakout NNNI 0123"
