File: Hardware/AD4630 breakout.kicad_pcb (KiCad board)
At the start: 4 copper layers, 35 x 40 mm, 26 parts, among them J1 IN0, J2 IN1, J4 IN0, U1 AD4630-24BBCZ, U2 AMS1117-1.8, U3 TXS0108EPW, U4 TXS0108EPW, U6 LTC6655

Commit message: updated files
Parts:
- added J3: IO, Connector_PinHeader_2.00mm:PinHeader_1x05_P2.00mm_Vertical, F.Cu at (127.0, 77.0)
- added J5: IO, Connector_PinHeader_2.00mm:PinHeader_1x05_P2.00mm_Vertical, F.Cu at (137.0, 75.0)
- added J6: IO, Connector_PinHeader_2.00mm:PinHeader_1x05_P2.00mm_Vertical, F.Cu at (157.0, 77.0)
- added J7: IO, Connector_PinHeader_2.00mm:PinHeader_1x05_P2.00mm_Vertical, F.Cu at (147.0, 75.0)
- added kibuzzard-63D190C6: G***, kibuzzard-63D190C6, F.Cu at (130.0, 77.0)
- added kibuzzard-63D19151: G***, kibuzzard-63D19151, F.Cu at (129.9, 79.0)
- added kibuzzard-63D191A1: G***, kibuzzard-63D191A1, F.Cu at (129.4, 81.0)
- added kibuzzard-63D1920D: G***, kibuzzard-63D1920D, F.Cu at (129.4, 83.0)
- moved C2 22.5 mm to (139.0, 81.0), turned to 135 degrees
- moved C3 19.3 mm to (145.0, 81.0), turned to -135 degrees
- moved C4 16.9 mm to (133.3, 87.2), turned to -45 degrees
- moved C1 13.9 mm to (150.8, 87.2), turned to 45 degrees
- moved U3 4.24 mm to (136.0, 84.0)
- moved U4 4.24 mm to (148.0, 84.0)
Connections:
- U3 pad 1: unconnected-(U3-Pad1) -> /CNV
- U3 pad 12: unconnected-(U3-Pad12) -> /NC
- U3 pad 3: unconnected-(U3-Pad3) -> /RST
- U3 pad 4: unconnected-(U3-Pad4) -> /SDO3
- U3 pad 5: unconnected-(U3-Pad5) -> /SDO1
- U3 pad 6: unconnected-(U3-Pad6) -> /SDO2
- U3 pad 7: unconnected-(U3-Pad7) -> /SDO0
- U3 pad 8: unconnected-(U3-Pad8) -> /SCK OUT
- U4 pad 12: unconnected-(U4-Pad12) -> /NC1
- U4 pad 3: unconnected-(U4-Pad3) -> /SDO4
- U4 pad 4: unconnected-(U4-Pad4) -> /SDO6
- U4 pad 5: unconnected-(U4-Pad5) -> /SDO5
- U4 pad 6: unconnected-(U4-Pad6) -> /SDO7
- U4 pad 7: unconnected-(U4-Pad7) -> /SCK
- U4 pad 8: unconnected-(U4-Pad8) -> /SDI
- U4 pad 9: unconnected-(U4-Pad9) -> /CS
Routing:
- net /SCK OUT: track 2.80 -> 9.66 mm
- net /SDO0: track 2.80 -> 9.06 mm
- net /SDO4: track 2.80 -> 9.00 mm
- net /SDO2: track 3.87 -> 9.69 mm
- net /SDO6: track 3.77 -> 9.53 mm
- net /NC1: track 0.00 -> 5.61 mm
- net /NC: track 0.00 -> 5.61 mm
- net /SDO1: track 2.90 -> 8.29 mm
- net /SDO5: track 2.80 -> 8.13 mm
- net /SDO3: track 3.77 -> 8.72 mm
- net /SDO7: track 3.77 -> 8.66 mm
- net /RST: track 3.77 -> 8.12 mm
- net /SCK: track 3.77 -> 8.06 mm
- net GND: track 7.99 -> 3.89 mm, vias 19 -> 15
- net /SDI: track 4.73 -> 8.59 mm
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- removed copper zone on F.Cu, net /REFIN
Other:
- board size 35 x 40 mm -> 30 x 40 mm

Commit message: updated files
Parts:
- removed kibuzzard-63D190C6: G***, kibuzzard-63D190C6
- removed kibuzzard-63D19151: G***, kibuzzard-63D19151
- removed kibuzzard-63D191A1: G***, kibuzzard-63D191A1
- removed kibuzzard-63D1920D: G***, kibuzzard-63D1920D
- added JP1: REFSEL, Jumper:SolderJumper-3_P1.3mm_Open_RoundedPad1.0x1.5mm, F.Cu at (132.2, 104.0)
- J1, J2, J4: footprint Connector_PinHeader_2.54mm:PinHeader_1x02_P2.54mm_Vertical -> Connector_PinHeader_2.00mm:PinHeader_1x02_P2.00mm_Vertical
- moved C14 28.3 mm to (133.0, 99.4), turned to 0 degrees
- moved U6 26.8 mm to (133.5, 96.0), turned to -90 degrees
- moved C13 26.2 mm to (133.0, 92.6), turned to 180 degrees
- moved C11 21.9 mm to (151.1, 92.8)
- moved C12 21.9 mm to (151.1, 99.2)
- moved U2 21.9 mm to (150.3, 96.0)
- moved J4 7.30 mm to (132.2, 107.8), turned to 90 degrees
- moved J2 7.01 mm to (144.2, 107.8)
- moved J1 7.00 mm to (137.7, 107.8)
- moved R2 4.21 mm to (139.7, 104.0)
- moved R4 4.20 mm to (146.2, 104.0)
- moved R3 4.20 mm to (144.2, 104.0)
- moved C5 4.20 mm to (138.7, 101.8)
- moved R1 4.20 mm to (137.7, 104.0)
- moved C6 4.20 mm to (145.2, 101.8)
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Connections:
- C14 pad 1: /REFIN -> /REFOUT
- J4 pad 1: /REFIN -> /REFEXT
- U6 pad 6: /REFIN -> /REFOUT
- U6 pad 7: /REFIN -> /REFOUT
Routing:
- net /SDO6/: track 6.70 -> 0.00 mm
- net /CNV/: track 6.70 -> 0.00 mm
- net /IN1-: track 9.92 -> 3.79 mm
- net /IN1+: track 10.0 -> 3.88 mm
- net /IN0+: track 9.94 -> 3.83 mm
- net /IN0-: track 10.0 -> 3.92 mm
- net /REFOUT: track 0.00 -> 4.67 mm
- net GND: track 3.89 -> 7.99 mm
- net Net-(J2-Pad2): track 5.80 -> 2.97 mm
- net Net-(J2-Pad1): track 5.80 -> 2.97 mm
- net Net-(J1-Pad2): track 5.80 -> 2.97 mm
- net Net-(J1-Pad1): track 5.80 -> 2.97 mm
- net /SDO2: track 9.69 -> 7.58 mm
- net /SDO1: track 8.29 -> 6.18 mm
- net /REFEXT: track 0.00 -> 2.03 mm
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- removed copper zone on F.Cu, net +5V
- removed copper zone on F.Cu, net Net-(C13-Pad1)
Other:
- board size 30 x 40 mm -> 27 x 30 mm
- board text added: "AD4630 Dev NNNI 0423"
- board text removed: "3V3"
- board text removed: "5V"
- board text removed: "AD4630 Breakout NNNI 0123"
- board text removed: "CKO"
- board text removed: "CNV"
- board text removed: "CS"
- board text removed: "DO0"
- board text removed: "DO1"
- board text removed: "DO2"
- board text removed: "DO3"
- board text removed: "DO4"
- board text removed: "DO5"
- board text removed: "DO6"
- board text removed: "DO7"
- board text removed: "GND"
- board text removed: "IN0+"
- board text removed: "IN0-"
- board text removed: "IN1+"
- board text removed: "IN1-"
- board text removed: "REF IN"
- board text removed: "RST"
- board text removed: "SCK"
- board text removed: "SDI"

Commit message: updated files
Parts:
- added H1: MountingHole, MountingHole:MountingHole_3.2mm_M3_Pad_Via, F.Cu at (120.8, 74.5)
- added H2: MountingHole, MountingHole:MountingHole_3.2mm_M3_Pad_Via, F.Cu at (161.8, 74.5)
- added H3: MountingHole, MountingHole:MountingHole_3.2mm_M3_Pad_Via, F.Cu at (120.8, 135.5)
- added H4: MountingHole, MountingHole:MountingHole_3.2mm_M3_Pad_Via, F.Cu at (161.8, 135.5)
- added U5: Elite-C, Keebio-Parts:Elite-C-castellated-29pin-holes, F.Cu at (141.3, 86.5)
- moved C1 75.4 mm to (81.3, 122.8)
- moved C4 75.4 mm to (66.8, 122.8)
- moved U2 75.4 mm to (82.3, 128.8)
- moved C2 75.4 mm to (72.5, 116.5)
- moved C3 75.4 mm to (75.5, 116.5)
- moved J3 75.4 mm to (60.5, 112.5)
- moved J4 75.4 mm to (64.2, 140.6)
- moved J5 75.4 mm to (70.5, 110.5)
- moved J6 75.4 mm to (87.5, 112.5)
- moved J7 75.4 mm to (77.5, 110.5)
- moved U6 75.4 mm to (65.5, 128.8)
- moved C11 75.4 mm to (83.2, 125.5)
- moved C12 75.4 mm to (83.2, 131.9)
- moved C13 75.4 mm to (65.0, 125.3)
- moved C14 75.4 mm to (65.0, 132.2)
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Other:
- board size 27 x 30 mm -> 50 x 70 mm
