File: Hardware/AD4630 breakout.kicad_sch (KiCad schematic)
At the start: 27 parts, among them J1 IN0, J2 IN1, J3 IO, J4 IN0, U1 AD4630-24BBCZ, U2 AMS1117-1.8, U3 TXS0108EPW, U4 TXS0108EPW, U6 LTC6655

Commit message: updated files
Parts:
- removed J3: IO, Connector_PinHeader_2.54mm:PinHeader_2x09_P2.54mm_Vertical, symbol Connector_Generic:Conn_02x09_Counter_Clockwise
Connections:
- net CNV: no longer U3.1 (A1)
- net CS: no longer U4.8 (A7)
- net RST: no longer U3.3 (A2)
- net SCK: no longer U4.6 (A5)
- net SCK OUT: no longer U3.8 (A7)
- net SDI: no longer U4.7 (A6)
- net SDO0: no longer U3.6 (A5)
- net SDO1: no longer U3.4 (A3)
- net SDO2: no longer U3.7 (A6)
- net SDO3: no longer U3.5 (A4)
- net SDO4: no longer U4.3 (A2)
- net SDO5: no longer U4.5 (A4)
- net SDO6: no longer U4.1 (A1)
- net SDO7: no longer U4.4 (A3)
Changed lines of the file:
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@@
-    (stroke (width 0) (type default) (color 0 0 0 0))
-  )
-  (wire (pts (xy 167.64 137.16) (xy 189.23 137.16))
     (stroke (width 0) (type default) (color 0 0 0 0))
   )
@@
     (stroke (width 0) (type default) (color 0 0 0 0))
   )
-  (wire (pts (xy 167.64 132.08) (xy 194.31 132.08))
+  (wire (pts (xy 167.64 104.14) (xy 177.8 104.14))
     (stroke (width 0) (type default) (color 0 0 0 0))
   )
@@
     (stroke (width 0) (type default) (color 0 0 0 0))
   )
-  (wire (pts (xy 167.64 134.62) (xy 191.77 134.62))
-    (stroke (width 0) (type default) (color 0 0 0 0))
-  )
   (wire (pts (xy 222.25 49.53) (xy 222.25 52.07))
     (stroke (width 0) (type default) (color 0 0 0 0))
@@
     (stroke (width 0) (type default) (color 0 0 0 0))
   )
-  (wire (pts (xy 167.64 124.46) (xy 201.93 124.46))
-    (stroke (width 0) (type default) (color 0 0 0 0))
-  )
   (polyline (pts (xy 165.1 189.23) (xy 165.1 228.6))
     (stroke (width 0) (type default) (color 0 0 0 0))
   )
-  (wire (pts (xy 167.64 121.92) (xy 204.47 121.92))
-    (stroke (width 0) (type default) (color 0 0 0 0))
-  )
   (wire (pts (xy 334.01 110.49) (xy 331.47 110.49))
     (stroke (width 0) (type default) (color 0 0 0 0))
@@
     (stroke (width 0) (type default) (color 0 0 0 0))
   )
+  (wire (pts (xy 167.64 127) (xy 177.8 127))
+    (stroke (width 0) (type default) (color 0 0 0 0))
+  )
   (wire (pts (xy 170.18 86.36) (xy 170.18 88.9))
     (stroke (width 0) (type default) (color 0 0 0 0))
   )
-  (wire (pts (xy 167.64 111.76) (xy 199.39 111.76))
-    (stroke (width 0) (type default) (color 0 0 0 0))
-  )
   (wire (pts (xy 59.69 107.95) (xy 64.77 107.95))
     (stroke (width 0) (type default) (color 0 0 0 0))
   )
+  (wire (pts (xy 167.64 132.08) (xy 177.8 132.08))
+    (stroke (width 0) (type default) (color 0 0 0 0))
+  )
   (wire (pts (xy 189.23 217.17) (xy 189.23 214.63))
     (stroke (width 0) (type default) (color 0 0 0 0))
@@
     (stroke (width 0) (type default) (color 0 0 0 0))
   )
+  (wire (pts (xy 167.64 114.3) (xy 177.8 114.3))
+    (stroke (width 0) (type default) (color 0 0 0 0))
+  )
   (wire (pts (xy 250.19 82.55) (xy 265.43 82.55))
     (stroke (width 0) (type default) (color 0 0 0 0))
@@
     (stroke (width 0) (type default) (color 0 0 0 0))
   )
+  (wire (pts (xy 167.64 109.22) (xy 177.8 109.22))
+    (stroke (width 0) (type default) (color 0 0 0 0))
+  )
   (wire (pts (xy 331.47 80.01) (xy 331.47 82.55))
     (stroke (width 0) (type default) (color 0 0 0 0))
@@
     (stroke (width 0) (type default) (color 0 0 0 0))
   )
+  (wire (pts (xy 167.64 111.76) (xy 177.8 111.76))
+    (stroke (width 0) (type default) (color 0 0 0 0))
+  )
   (wire (pts (xy 74.93 91.44) (xy 77.47 91.44))
     (stroke (width 0) (type default) (color 0 0 0 0))
@@
     (stroke (width 0) (type default) (color 0 0 0 0))
   )
+  (wire (pts (xy 167.64 124.46) (xy 177.8 124.46))
+    (stroke (width 0) (type default) (color 0 0 0 0))
+  )
   (polyline (pts (xy 223.52 189.23) (xy 190.5 189.23))
     (stroke (width 0) (type default) (color 0 0 0 0))
@@
     (stroke (width 0) (type default) (color 0 0 0 0))
   )
+  (wire (pts (xy 167.64 101.6) (xy 177.8 101.6))
+    (stroke (width 0) (type default) (color 0 0 0 0))
+  )
   (wire (pts (xy 331.47 125.73) (xy 331.47 128.27))
     (stroke (width 0) (type default) (color 0 0 0 0))
   )
-  (wire (pts (xy 167.64 129.54) (xy 196.85 129.54))
-    (stroke (width 0) (type default) (color 0 0 0 0))
-  )
   (wire (pts (xy 331.47 105.41) (xy 331.47 107.95))
     (stroke (width 0) (type default) (color 0 0 0 0))
@@
     (stroke (width 0) (type default) (color 0 0 0 0))
   )
-  (wire (pts (xy 167.64 101.6) (xy 189.23 101.6))
-    (stroke (width 0) (type default) (color 0 0 0 0))
-  )
   (wire (pts (xy 270.51 77.47) (xy 250.19 77.47))
     (stroke (width 0) (type default) (color 0 0 0 0))
@@
     (stroke (width 0) (type default) (color 0 0 0 0))
   )
+  (wire (pts (xy 167.64 129.54) (xy 177.8 129.54))
+    (stroke (width 0) (type default) (color 0 0 0 0))
+  )
   (wire (pts (xy 255.27 92.71) (xy 250.19 92.71))
     (stroke (width 0) (type default) (color 0 0 0 0))
@@
     (stroke (width 0) (type default) (color 0 0 0 0))
   )
+  (wire (pts (xy 167.64 121.92) (xy 177.8 121.92))
+    (stroke (width 0) (type default) (color 0 0 0 0))
+  )
   (wire (pts (xy 252.73 190.5) (xy 252.73 193.04))
     (stroke (width 0) (type default) (color 0 0 0 0))
@@
     (stroke (width 0) (type default) (color 0 0 0 0))
   )
-  (wire (pts (xy 167.64 116.84) (xy 204.47 116.84))
+  (wire (pts (xy 167.64 116.84) (xy 177.8 116.84))
     (stroke (width 0) (type default) (color 0 0 0 0))
   )
@@
     (stroke (width 0) (type default) (color 0 0 0 0))
   )
+  (wire (pts (xy 167.64 137.16) (xy 177.8 137.16))
+    (stroke (width 0) (type default) (color 0 0 0 0))
+  )
+  (wire (pts (xy 167.64 134.62) (xy 177.8 134.62))
+    (stroke (width 0) (type default) (color 0 0 0 0))
+  )
   (wire (pts (xy 229.87 149.86) (xy 260.35 149.86))
     (stroke (width 0) (type default) (color 0 0 0 0))
@@
     (stroke (width 0) (type default) (color 0 0 0 0))
   )
-  (wire (pts (xy 167.64 127) (xy 199.39 127))
-    (stroke (width 0) (type default) (color 0 0 0 0))
-  )
   (wire (pts (xy 77.47 91.44) (xy 77.47 83.82))
     (stroke (width 0) (type default) (color 0 0 0 0))
@@
     (stroke (width 0) (type default) (color 0 0 0 0))
   )
-  (wire (pts (xy 167.64 109.22) (xy 196.85 109.22))
-    (stroke (width 0) (type default) (color 0 0 0 0))
-  )
   (wire (pts (xy 201.93 90.17) (xy 209.55 90.17))
     (stroke (width 0) (type default) (color 0 0 0 0))
@@
     (stroke (width 0) (type default) (color 0 0 0 0))
   )
-  (wire (pts (xy 167.64 114.3) (xy 201.93 114.3))
-    (stroke (width 0) (type default) (color 0 0 0 0))
-  )
   (wire (pts (xy 252.73 182.88) (xy 252.73 185.42))
     (stroke (width 0) (type default) (color 0 0 0 0))
@@
     (stroke (width 0) (type default) (color 0 0 0 0))
   )
-  (wire (pts (xy 167.64 106.68) (xy 194.31 106.68))
-    (stroke (width 0) (type default) (color 0 0 0 0))
-  )
   (wire (pts (xy 222.25 119.38) (xy 222.25 134.62))
     (stroke (width 0) (type default) (color 0 0 0 0))
@@
     (stroke (width 0) (type default) (color 0 0 0 0))
   )
-  (wire (pts (xy 167.64 104.14) (xy 191.77 104.14))
-    (stroke (width 0) (type default) (color 0 0 0 0))
-  )
   (wire (pts (xy 326.39 168.91) (xy 326.39 166.37))
     (stroke (width 0) (type default) (color 0 0 0 0))
   )
   (wire (pts (xy 209.55 154.94) (xy 194.31 154.94))
+    (stroke (width 0) (type default) (color 0 0 0 0))
+  )
+  (wire (pts (xy 167.64 106.68) (xy 177.8 106.68))
     (stroke (width 0) (type default) (color 0 0 0 0))
   )
@@
     (pin "1")
     (pin "2")
-  )
-  (symbol (lib_id "Connector_Generic:Conn_02x09_Counter_Clockwise") (at 242.57 87.63 0) (unit 1)
-    (in_bom yes) (on_board yes)
-    (property "Reference" "J3" (id 0) (at 243.84 71.12 0))
-    (property "Value" "IO" (id 1) (at 243.84 73.66 0))
-    (property "Footprint" "Connector_PinHeader_2.54mm:PinHeader_2x09_P2.54mm_Vertical" (id 2) (at 242.57 87.63 0)
-      (effects (font (size 1.27 1.27)) hide)
-    )
-    (property "Datasheet" "~" (id 3) (at 242.57 87.63 0)
-      (effects (font (size 1.27 1.27)) hide)
-    )
-    (pin "1")
-    (pin "10")
-    (pin "11")
-    (pin "12")
-    (pin "13")
-    (pin "14")
-    (pin "15")
-    (pin "16")
-    (pin "17")
-    (pin "18")
-    (pin "2")
-    (pin "3")
-    (pin "4")
-    (pin "5")
-    (pin "6")
-    (pin "7")
-    (pin "8")
-    (pin "9")
   )
   (symbol (lib_id "power:GND") (at 226.06 129.54 0) (unit 1)
@@
       (reference "J2") (unit 1) (value "IN1") (footprint "Connector_PinHeader_2.54mm:PinHeader_1x02_P2.54mm_Vertical")
     )
-    (path "/0fa67205-a6e8-49d2-947c-4edf57faf2dd"
-      (reference "J3") (unit 1) (value "IO") (footprint "Connector_PinHeader_2.54mm:PinHeader_2x09_P2.54mm_Vertical")
-    )
     (path "/f595fc96-6462-4dba-95d3-e7369442b29b"

Commit message: updated files
Parts:
- added J3, J5, J6, J7: IO, Connector_PinHeader_2.00mm:PinHeader_1x05_P2.00mm_Vertical, symbol Connector_Generic:Conn_01x05
Connections:
- net +3V3: now also J3.4 (Pin_4), J7.2 (Pin_2)
- net CNV: now also U3.1 (A1)
- net CNV/: now also J3.5 (Pin_5)
- net CS: now also U4.9 (A8)
- net CS/: now also J6.3 (Pin_3)
- net GND: now also J5.1 (Pin_1), J6.5 (Pin_5)
- net RST: now also U3.3 (A2)
- net RST/: now also J3.3 (Pin_3)
- net SCK: now also U4.7 (A6)
- net SCK OUT: now also U3.8 (A7)
- net SCKo/: now also J5.3 (Pin_3)
- net SCK/: now also J6.1 (Pin_1)
- net SDI: now also U4.8 (A7)
- net SDI/: now also J6.2 (Pin_2)
- net SDO0: now also U3.7 (A6)
- net SDO0/: now also J5.5 (Pin_5)
- net SDO1: now also U3.5 (A4)
- net SDO1/: now also J3.2 (Pin_2)
- net SDO2: now also U3.6 (A5)
- net SDO2/: now also J5.4 (Pin_4)
- net SDO3: now also U3.4 (A3)
- net SDO3/: now also J3.1 (Pin_1)
- net SDO4: now also U4.3 (A2)
- net SDO4/: now also J7.3 (Pin_3)
- net SDO5: now also U4.5 (A4)
- net SDO5/: now also J7.5 (Pin_5)
- net SDO6: now also U4.4 (A3)
- net SDO6/: now also J7.1 (Pin_1)
- net SDO7: now also U4.6 (A5)
- net SDO7/: now also J7.4 (Pin_4)
- net NC1: now reaches U4.12 (B8)
- net NC1: now also J6.4 (Pin_4)
- net NC: now reaches U3.12 (B8)
- net NC: now also J5.2 (Pin_2)
- no-connect marks 4 -> 2

Commit message: updated files
Parts:
- added JP1: REFSEL, Jumper:SolderJumper-3_P1.3mm_Open_RoundedPad1.0x1.5mm, symbol Jumper:SolderJumper_3_Open
- J1, J2, J4: footprint Connector_PinHeader_2.54mm:PinHeader_1x02_P2.54mm_Vertical -> Connector_PinHeader_2.00mm:PinHeader_1x02_P2.00mm_Vertical
Connections:
- net REFIN: now also JP1.2 (C); no longer C14.1, J4.1 (Pin_1), U6.6 (VOUT_S), U6.7 (VOUT_F)
- new net REFEXT: J4.1 (Pin_1), JP1.3 (B)
- new net REFOUT: C14.1, JP1.1 (A), U6.6 (VOUT_S), U6.7 (VOUT_F)
Other:
- moved on the sheet: J4
Changed lines of the file:
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@@
   (junction (at 328.93 64.77) (diameter 0) (color 0 0 0 0)
   )
-  (junction (at 214.63 199.39) (diameter 0) (color 0 0 0 0)
-  )
   (junction (at 328.93 62.23) (diameter 0) (color 0 0 0 0)
   )
@@
   )
   (junction (at 331.47 87.63) (diameter 0) (color 0 0 0 0)
-  )
-  (junction (at 214.63 217.17) (diameter 0) (color 0 0 0 0)
   )
   (junction (at 93.98 106.68) (diameter 0) (color 0 0 0 0)
@@
   (no_connect (at 209.55 95.25))
   (no_connect (at 209.55 144.78))
-  (wire (pts (xy 233.68 208.28) (xy 231.14 208.28))
-    (stroke (width 0) (type default) (color 0 0 0 0))
-  )
   (wire (pts (xy 170.18 93.98) (xy 177.8 93.98))
     (stroke (width 0) (type default) (color 0 0 0 0))
@@
     (stroke (width 0) (type default) (color 0 0 0 0))
   )
+  (wire (pts (xy 154.94 175.26) (xy 157.48 175.26))
+    (stroke (width 0) (type default) (color 0 0 0 0))
+  )
   (wire (pts (xy 334.01 130.81) (xy 331.47 130.81))
     (stroke (width 0) (type default) (color 0 0 0 0))
@@
     (stroke (width 0) (type default) (color 0 0 0 0))
   )
-  (wire (pts (xy 231.14 205.74) (xy 233.68 205.74))
-    (stroke (width 0) (type default) (color 0 0 0 0))
-  )
   (wire (pts (xy 222.25 52.07) (xy 222.25 67.31))
     (stroke (width 0) (type default) (color 0 0 0 0))
   )
+  (wire (pts (xy 149.86 180.34) (xy 142.24 180.34))
+    (stroke (width 0) (type default) (color 0 0 0 0))
+  )
   (wire (pts (xy 331.47 72.39) (xy 331.47 74.93))
     (stroke (width 0) (type default) (color 0 0 0 0))
@@
     (stroke (width 0) (type default) (color 0 0 0 0))
   )
+  (wire (pts (xy 142.24 180.34) (xy 142.24 176.53))
+    (stroke (width 0) (type default) (color 0 0 0 0))
+  )
   (wire (pts (xy 331.47 77.47) (xy 331.47 80.01))
     (stroke (width 0) (type default) (color 0 0 0 0))
@@
     (stroke (width 0) (type default) (color 0 0 0 0))
   )
-  (wire (pts (xy 214.63 217.17) (xy 231.14 217.17))
-    (stroke (width 0) (type default) (color 0 0 0 0))
-  )
   (wire (pts (xy 331.47 74.93) (xy 334.01 74.93))
     (stroke (width 0) (type default) (color 0 0 0 0))
@@
     (stroke (width 0) (type default) (color 0 0 0 0))
   )
+  (wire (pts (xy 154.94 175.26) (xy 154.94 177.8))
+    (stroke (width 0) (type default) (color 0 0 0 0))
+  )
   (wire (pts (xy 64.77 91.44) (xy 67.31 91.44))
     (stroke (width 0) (type default) (color 0 0 0 0))
@@
     (stroke (width 0) (type default) (color 0 0 0 0))
   )
-  (wire (pts (xy 214.63 199.39) (xy 231.14 199.39))
-    (stroke (width 0) (type default) (color 0 0 0 0))
-  )
   (wire (pts (xy 217.17 134.62) (xy 217.17 119.38))
     (stroke (width 0) (type default) (color 0 0 0 0))
@@
     (stroke (width 0) (type default) (color 0 0 0 0))
   )
+  (wire (pts (xy 128.27 172.72) (xy 137.16 172.72))
+    (stroke (width 0) (type default) (color 0 0 0 0))
+  )
   (wire (pts (xy 252.73 190.5) (xy 252.73 193.04))
     (stroke (width 0) (type default) (color 0 0 0 0))
@@
     (stroke (width 0) (type default) (color 0 0 0 0))
   )
-  (wire (pts (xy 231.14 208.28) (xy 231.14 217.17))
-    (stroke (width 0) (type default) (color 0 0 0 0))
-  )
   (wire (pts (xy 290.83 49.53) (xy 290.83 54.61))
     (stroke (width 0) (type default) (color 0 0 0 0))
@@
     (stroke (width 0) (type default) (color 0 0 0 0))
   )
+  (wire (pts (xy 147.32 172.72) (xy 157.48 172.72))
+    (stroke (width 0) (type default) (color 0 0 0 0))
+  )
   (wire (pts (xy 170.18 93.98) (xy 167.64 93.98))
     (stroke (width 0) (type default) (color 0 0 0 0))
@@
     (stroke (width 0) (type default) (color 0 0 0 0))
   )
-  (wire (pts (xy 231.14 199.39) (xy 231.14 205.74))
-    (stroke (width 0) (type default) (color 0 0 0 0))
-  )
   (wire (pts (xy 331.47 146.05) (xy 334.01 146.05))
     (stroke (width 0) (type default) (color 0 0 0 0))
@@
     (effects (font (size 1.27 1.27)) (justify right bottom))
   )
+  (label "REFEXT" (at 156.21 172.72 180)
+    (effects (font (size 1.27 1.27)) (justify right bottom))
+  )
   (label "RST" (at 200.66 80.01 0)
     (effects (font (size 1.27 1.27)) (justify left bottom))
@@
     (effects (font (size 1.27 1.27)) (justify right bottom))
   )
+  (label "REFOUT" (at 128.27 172.72 0)
+    (effects (font (size 1.27 1.27)) (justify left bottom))
+  )
   (label "CNV{slash}" (at 237.49 77.47 180)
     (effects (font (size 1.27 1.27)) (justify right bottom))
@@
     (effects (font (size 1.27 1.27)) (justify left bottom))
   )
-  (label "REFIN" (at 214.63 199.39 180)
+  (label "REFOUT" (at 214.63 199.39 180)
     (effects (font (size 1.27 1.27)) (justify right bottom))
   )
@@
   (label "CNV" (at 200.66 77.47 0)
     (effects (font (size 1.27 1.27)) (justify left bottom))
+  )
+  (label "REFIN" (at 149.86 180.34 180)
+    (effects (font (size 1.27 1.27)) (justify right bottom))
   )
   (label "REFIN" (at 177.8 96.52 180)
@@
     (property "Reference" "J1" (id 0) (at 54.61 73.66 0))
     (property "Value" "IN0" (id 1) (at 54.61 76.2 0))
-    (property "Footprint" "Connector_PinHeader_2.54mm:PinHeader_1x02_P2.54mm_Vertical" (id 2) (at 54.61 80.01 0)
+    (property "Footprint" "Connector_PinHeader_2.00mm:PinHeader_1x02_P2.00mm_Vertical" (id 2) (at 54.61 80.01 0)
       (effects (font (size 1.27 1.27)) hide)
     )
@@
     )
     (property "Datasheet" "" (id 3) (at 222.25 116.84 0)
+      (effects (font (size 1.27 1.27)) hide)
+    )
+    (pin "1")
+  )
+  (symbol (lib_id "power:GND") (at 154.94 177.8 0) (unit 1)
+    (in_bom yes) (on_board yes)
+    (property "Reference" "#PWR0114" (id 0) (at 154.94 184.15 0)
+      (effects (font (size 1.27 1.27)) hide)
+    )
+    (property "Value" "GND" (id 1) (at 154.94 182.88 0))
+    (property "Footprint" "" (id 2) (at 154.94 177.8 0)
+      (effects (font (size 1.27 1.27)) hide)
+    )
+    (property "Datasheet" "" (id 3) (at 154.94 177.8 0)
       (effects (font (size 1.27 1.27)) hide)
     )
@@
     (property "Reference" "J2" (id 0) (at 54.61 99.06 0))
     (property "Value" "IN1" (id 1) (at 54.61 101.6 0))
-    (property "Footprint" "Connector_PinHeader_2.54mm:PinHeader_1x02_P2.54mm_Vertical" (id 2) (at 54.61 105.41 0)
+    (property "Footprint" "Connector_PinHeader_2.00mm:PinHeader_1x02_P2.00mm_Vertical" (id 2) (at 54.61 105.41 0)
       (effects (font (size 1.27 1.27)) hide)
     )
@@
     (pin "1")
     (pin "2")
+  )
+  (symbol (lib_id "Jumper:SolderJumper_3_Open") (at 142.24 172.72 0) (unit 1)
+    (in_bom yes) (on_board yes)
+    (property "Reference" "JP1" (id 0) (at 142.24 166.37 0))
+    (property "Value" "REFSEL" (id 1) (at 142.24 168.91 0))
+    (property "Footprint" "Jumper:SolderJumper-3_P1.3mm_Open_RoundedPad1.0x1.5mm" (id 2) (at 142.24 172.72 0)
+      (effects (font (size 1.27 1.27)) hide)
+    )
+    (property "Datasheet" "~" (id 3) (at 142.24 172.72 0)
+      (effects (font (size 1.27 1.27)) hide)
+    )
+    (pin "1")
+    (pin "2")
+    (pin "3")
   )
   (symbol (lib_id "power:GND") (at 219.71 172.72 0) (unit 1)
@@
     (pin "1")
   )
-  (symbol (lib_id "Connector_Generic:Conn_01x02") (at 238.76 205.74 0) (unit 1)
-    (in_bom yes) (on_board yes)
-    (property "Reference" "J4" (id 0) (at 238.76 199.39 0))
-    (property "Value" "IN0" (id 1) (at 238.76 201.93 0))
-    (property "Footprint" "Connector_PinHeader_2.54mm:PinHeader_1x02_P2.54mm_Vertical" (id 2) (at 238.76 205.74 0)
-      (effects (font (size 1.27 1.27)) hide)
-    )
-    (property "Datasheet" "~" (id 3) (at 238.76 205.74 0)
+  (symbol (lib_id "Connector_Generic:Conn_01x02") (at 162.56 172.72 0) (unit 1)
+    (in_bom yes) (on_board yes)
+    (property "Reference" "J4" (id 0) (at 162.56 166.37 0))
+    (property "Value" "IN0" (id 1) (at 162.56 168.91 0))
+    (property "Footprint" "Connector_PinHeader_2.00mm:PinHeader_1x02_P2.00mm_Vertical" (id 2) (at 162.56 172.72 0)
+      (effects (font (size 1.27 1.27)) hide)
+    )
+    (property "Datasheet" "~" (id 3) (at 162.56 172.72 0)
       (effects (font (size 1.27 1.27)) hide)
     )
@@
       (reference "#PWR0113") (unit 1) (value "+3.3V") (footprint "")
     )
+    (path "/2a936565-e6e2-475e-aa57-3ce2cebb6b1e"
+      (reference "#PWR0114") (unit 1) (value "GND") (footprint "")
+    )
     (path "/a295f9c6-a14c-45bc-bb07-450dff44d677"
       (reference "C1") (unit 1) (value "10uF") (footprint "Capacitor_SMD:C_0603_1608Metric")
@@
     )
     (path "/260f89fb-b1fb-4c40-993e-488233ad044e"
-      (reference "J1") (unit 1) (value "IN0") (footprint "Connector_PinHeader_2.54mm:PinHeader_1x02_P2.54mm_Vertical")
+      (reference "J1") (unit 1) (value "IN0") (footprint "Connector_PinHeader_2.00mm:PinHeader_1x02_P2.00mm_Vertical")
     )
     (path "/e01a2577-48b9-434e-89c8-6ca8fb34a23a"
-      (reference "J2") (unit 1) (value "IN1") (footprint "Connector_PinHeader_2.54mm:PinHeader_1x02_P2.54mm_Vertical")
+      (reference "J2") (unit 1) (value "IN1") (footprint "Connector_PinHeader_2.00mm:PinHeader_1x02_P2.00mm_Vertical")
     )
     (path "/9400265f-d3ba-492a-9aec-1408f87d5024"
@@
     )
     (path "/f595fc96-6462-4dba-95d3-e7369442b29b"
-      (reference "J4") (unit 1) (value "IN0") (footprint "Connector_PinHeader_2.54mm:PinHeader_1x02_P2.54mm_Vertical")
+      (reference "J4") (unit 1) (value "IN0") (footprint "Connector_PinHeader_2.00mm:PinHeader_1x02_P2.00mm_Vertical")
     )
     (path "/2f06a515-8992-4d6b-b5ab-0c38510475b8"
@@
       (reference "J7") (unit 1) (value "IO") (footprint "Connector_PinHeader_2.00mm:PinHeader_1x05_P2.00mm_Vertical")
     )
+    (path "/f02d95f9-5b6b-4846-a958-08f2f9419acb"
+      (reference "JP1") (unit 1) (value "REFSEL") (footprint "Jumper:SolderJumper-3_P1.3mm_Open_RoundedPad1.0x1.5mm")
+    )
     (path "/777b03c0-e8c0-401e-8d70-fcb07762e0c6"
