File: Hardware/AD4630 breakout.kicad_sch (KiCad schematic)
At the start: 31 parts, among them J1 IN0, J2 IN1, J3 IO, J4 IN0, J5 IO, J6 IO, J7 IO, U1 AD4630-24BBCZ, U2 AMS1117-1.8, U3 TXS0108EPW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

Commit message: updated files
Parts:
- added H1, H2, H3, H4: MountingHole, MountingHole:MountingHole_3.2mm_M3_Pad_Via, symbol Mechanical:MountingHole
- added U5: Elite-C, Keebio-Parts:Elite-C-castellated-29pin-holes, symbol keebio:Elite-C
Changed lines of the file:
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@@
     (pin "5")
+  )
+  (symbol (lib_id "Mechanical:MountingHole") (at 283.21 256.54 0) (unit 1)
+    (in_bom yes) (on_board yes)
+    (property "Reference" "H1" (id 0) (at 285.75 255.27 0)
+      (effects (font (size 1.27 1.27)) (justify left))
+    )
+    (property "Value" "MountingHole" (id 1) (at 285.75 257.81 0)
+      (effects (font (size 1.27 1.27)) (justify left))
+    )
+    (property "Footprint" "MountingHole:MountingHole_3.2mm_M3_Pad_Via" (id 2) (at 283.21 256.54 0)
+      (effects (font (size 1.27 1.27)) hide)
+    )
+    (property "Datasheet" "~" (id 3) (at 283.21 256.54 0)
+      (effects (font (size 1.27 1.27)) hide)
+    )
   )
   (symbol (lib_id "power:GND") (at 213.36 62.23 0) (unit 1)
@@
     )
     (pin "1")
+  )
+  (symbol (lib_id "Mechanical:MountingHole") (at 283.21 269.24 0) (unit 1)
+    (in_bom yes) (on_board yes)
+    (property "Reference" "H3" (id 0) (at 285.75 267.97 0)
+      (effects (font (size 1.27 1.27)) (justify left))
+    )
+    (property "Value" "MountingHole" (id 1) (at 285.75 270.51 0)
+      (effects (font (size 1.27 1.27)) (justify left))
+    )
+    (property "Footprint" "MountingHole:MountingHole_3.2mm_M3_Pad_Via" (id 2) (at 283.21 269.24 0)
+      (effects (font (size 1.27 1.27)) hide)
+    )
+    (property "Datasheet" "~" (id 3) (at 283.21 269.24 0)
+      (effects (font (size 1.27 1.27)) hide)
+    )
   )
   (symbol (lib_id "Device:R") (at 71.12 71.12 90) (unit 1)
@@
     (pin "2")
   )
+  (symbol (lib_id "keebio:Elite-C") (at 73.66 176.53 0) (unit 1)
+    (in_bom yes) (on_board yes) (fields_autoplaced)
+    (property "Reference" "U5" (id 0) (at 73.66 154.94 0)
+      (effects (font (size 1.524 1.524)))
+    )
+    (property "Value" "Elite-C" (id 1) (at 73.66 158.75 0)
+      (effects (font (size 1.524 1.524)))
+    )
+    (property "Footprint" "Keebio-Parts:Elite-C-castellated-29pin-holes" (id 2) (at 100.33 240.03 90)
+      (effects (font (size 1.524 1.524)) hide)
+    )
+    (property "Datasheet" "" (id 3) (at 100.33 240.03 90)
+      (effects (font (size 1.524 1.524)) hide)
+    )
+    (pin "1")
+    (pin "10")
+    (pin "11")
+    (pin "12")
+    (pin "13")
+    (pin "14")
+    (pin "15")
+    (pin "16")
+    (pin "17")
+    (pin "18")
+    (pin "19")
+    (pin "2")
+    (pin "20")
+    (pin "21")
+    (pin "22")
+    (pin "23")
+    (pin "24")
+    (pin "25")
+    (pin "26")
+    (pin "27")
+    (pin "28")
+    (pin "29")
+    (pin "3")
+    (pin "4")
+    (pin "5")
+    (pin "6")
+    (pin "7")
+    (pin "8")
+    (pin "9")
+  )
   (symbol (lib_id "Regulator_Linear:AMS1117-1.8") (at 262.89 182.88 0) (unit 1)
     (in_bom yes) (on_board yes)
@@
     )
     (pin "1")
+  )
+  (symbol (lib_id "Mechanical:MountingHole") (at 283.21 262.89 0) (unit 1)
+    (in_bom yes) (on_board yes)
+    (property "Reference" "H2" (id 0) (at 285.75 261.62 0)
+      (effects (font (size 1.27 1.27)) (justify left))
+    )
+    (property "Value" "MountingHole" (id 1) (at 285.75 264.16 0)
+      (effects (font (size 1.27 1.27)) (justify left))
+    )
+    (property "Footprint" "MountingHole:MountingHole_3.2mm_M3_Pad_Via" (id 2) (at 283.21 262.89 0)
+      (effects (font (size 1.27 1.27)) hide)
+    )
+    (property "Datasheet" "~" (id 3) (at 283.21 262.89 0)
+      (effects (font (size 1.27 1.27)) hide)
+    )
   )
   (symbol (lib_id "Device:C_Small") (at 252.73 187.96 0) (mirror y) (unit 1)
@@
     (pin "5")
   )
+  (symbol (lib_id "Mechanical:MountingHole") (at 283.21 275.59 0) (unit 1)
+    (in_bom yes) (on_board yes)
+    (property "Reference" "H4" (id 0) (at 285.75 274.32 0)
+      (effects (font (size 1.27 1.27)) (justify left))
+    )
+    (property "Value" "MountingHole" (id 1) (at 285.75 276.86 0)
+      (effects (font (size 1.27 1.27)) (justify left))
+    )
+    (property "Footprint" "MountingHole:MountingHole_3.2mm_M3_Pad_Via" (id 2) (at 283.21 275.59 0)
+      (effects (font (size 1.27 1.27)) hide)
+    )
+    (property "Datasheet" "~" (id 3) (at 283.21 275.59 0)
+      (effects (font (size 1.27 1.27)) hide)
+    )
+  )
   (symbol (lib_id "Device:C_Small") (at 214.63 207.01 0) (unit 1)
     (in_bom yes) (on_board yes)
@@
       (reference "C14") (unit 1) (value "10uF") (footprint "Capacitor_SMD:C_0603_1608Metric")
     )
+    (path "/3b44024a-e554-45c2-9ec2-39a81d8ce35b"
+      (reference "H1") (unit 1) (value "MountingHole") (footprint "MountingHole:MountingHole_3.2mm_M3_Pad_Via")
+    )
+    (path "/ab53ae87-1fc6-4c79-b94d-99284134dc61"
+      (reference "H2") (unit 1) (value "MountingHole") (footprint "MountingHole:MountingHole_3.2mm_M3_Pad_Via")
+    )
+    (path "/762d1202-95a3-4fee-9943-e11b0a028d9e"
+      (reference "H3") (unit 1) (value "MountingHole") (footprint "MountingHole:MountingHole_3.2mm_M3_Pad_Via")
+    )
+    (path "/db625493-42be-4962-aa29-2e6dc8c9d4fa"
+      (reference "H4") (unit 1) (value "MountingHole") (footprint "MountingHole:MountingHole_3.2mm_M3_Pad_Via")
+    )
     (path "/260f89fb-b1fb-4c40-993e-488233ad044e"
       (reference "J1") (unit 1) (value "IN0") (footprint "Connector_PinHeader_2.00mm:PinHeader_1x02_P2.00mm_Vertical")
@@
       (reference "U4") (unit 1) (value "TXS0108EPW") (footprint "Package_SO:TSSOP-20_4.4x6.5mm_P0.65mm")
     )
+    (path "/872ee065-c3a6-4955-a12e-06cc96be8e73"
+      (reference "U5") (unit 1) (value "Elite-C") (footprint "Keebio-Parts:Elite-C-castellated-29pin-holes")
+    )
     (path "/d9e0b22e-a41d-439d-83b3-b78c2afa32c6"
